Commit message: MOD: added base_footprint to the robot urdf xacro

File: phantomx_reactor_arm_description/robots/phantomx_reactor_arm_4dof.urdf.xacro (robot description, xacro)
@@ -1,16 +1,15 @@
 <?xml version="1.0"?>
-<robot name="robospect" xmlns:xacro="http://www.ros.org/wiki/xacro">
-	<!-- Import Robospect Base -->
+<robot name="phantomx_reactor_arm" xmlns:xacro="http://www.ros.org/wiki/xacro">
+	<!-- Import URDF xacro model -->
 	<xacro:include filename="$(find phantomx_reactor_arm_description)/urdf/phantomx_reactor_4dof.urdf.xacro" />
 	<link name="base_footprint">
+		<visual>
+			<origin xyz="0 0 0" rpy="0 0 0"/>
+			<geometry>
+				<box size="0.001 0.001 0.001" />
+			</geometry>
+		</visual>
 	</link>
-	<joint name="base_footprint_joint" type="fixed">
-	 <origin xyz="0 0 0" rpy="0 0 0" />
-	 <parent link="base_footprint"/>
-	 <child link="base_link" />
-	</joint>
-	<link name="base_link">
-	</link>
-	<xacro:phantomx_reactor_4dof name="arm" parent="base_link">
+	<xacro:phantomx_reactor_4dof name="arm" parent="base_footprint">
 		<origin xyz="0 0 0" rpy="0 0 0" />
 	</xacro:phantomx_reactor_4dof>
