Commit message: description: unifying models for wrist version

File: phantomx_reactor_arm_description/robots/phantomx_reactor_arm_wrist.urdf.xacro (robot description, xacro)
@@ -11,6 +11,6 @@
 		</visual>
 	</link>
-	<xacro:phantomx_reactor_wrist prefix="arm_" parent="base_footprint">
+	<xacro:phantomx_reactor_wrist prefix="" parent="base_footprint">
 		<origin xyz="0 0 0" rpy="0 0 0" />
-	</xacro:phantomx_reactor_wrist		>
+	</xacro:phantomx_reactor_wrist>
 </robot>

File: phantomx_reactor_arm_description/urdf/phantomx_reactor_wrist.urdf.xacro (robot description, xacro)
@@ -2,12 +2,16 @@
 <robot name="phantomx_reactor" xmlns:xacro="http://www.ros.org/wiki/xacro">
 	<xacro:property name="PI" value="3.141593"/>
-	<xacro:property name="joint_1_upper_limit" value="${PI}"/>
-	<xacro:property name="joint_1_lower_limit" value="-${PI}"/>
-	<xacro:property name="joint_2_upper_limit" value="${PI/2}"/>
-	<xacro:property name="joint_2_lower_limit" value="-${PI/2}"/>
-	<xacro:property name="joint_3_upper_limit" value="1.8"/>
-	<xacro:property name="joint_3_lower_limit" value="-1.0"/>
-	<xacro:property name="joint_4_upper_limit" value="${PI/2}"/>
-	<xacro:property name="joint_4_lower_limit" value="-${PI/2}"/>
+	<xacro:property name="shoulder_yaw_joint_upper_limit" value="${PI}"/>
+	<xacro:property name="shoulder_yaw_joint_lower_limit" value="-${PI}"/>
+	<xacro:property name="shoulder_pitch_joint_upper_limit" value="${PI/2}"/>
+	<xacro:property name="shoulder_pitch_joint_lower_limit" value="-${PI/2}"/>
+	<xacro:property name="elbow_pitch_joint_upper_limit" value="${PI/2}"/>
+	<xacro:property name="elbow_pitch_joint_lower_limit" value="-${PI/2}"/>
+	<xacro:property name="wrist_pitch_upper_limit" value="1.9"/>
+	<xacro:property name="wrist_pitch_lower_limit" value="-1.7"/>
+	<xacro:property name="wrist_roll_upper_limit" value="${PI}"/>
+	<xacro:property name="wrist_roll_lower_limit" value="-${PI}"/>
+	<xacro:property name="gripper_joint_upper_limit" value="0.0"/>
+	<xacro:property name="gripper_joint_lower_limit" value="0.03"/>
 	<xacro:macro name="phantomx_reactor_wrist" params="parent prefix *origin">
 	    <!-- ARM BASE JOINT -->
@@ -42,13 +46,13 @@
 		</link>
 		<!-- SHOULDER YAW -->
-		<joint name="${prefix}1_joint" type="revolute">
+		<joint name="${prefix}shoulder_yaw_joint" type="revolute">
 			<origin xyz="0 0 0.081" rpy="0 0 0" />
+			<!--origin xyz="0 0 0.081" rpy="0 0 0" /-->
 			<parent link="${prefix}base_link" />
-			<child link="${prefix}1_link" />
+			<child link="${prefix}shoulder_link" />
 			<axis xyz="0 0 1" />
-			<limit effort="1.5" velocity="6.178465545" lower="-3.141593" upper="3.141593" />
-			<!--limit effort="1.5" velocity="6.178465545" lower="-2.57079632679" upper="2.57079632679" /-->
-		</joint>
-		<link name="${prefix}1_link">
+			<limit effort="1.5" velocity="6.178465545" lower="${shoulder_yaw_joint_lower_limit}" upper="${shoulder_yaw_joint_upper_limit}" />
+		</joint>
+		<link name="${prefix}shoulder_link">
 			<inertial>
 			  <origin xyz="5.5296E-07 0.00048339 0.0026355" rpy="0 0 0" />
@@ -74,12 +78,12 @@
 		</link>
 		<!-- SHOULDER PITCH -->
-		<joint name="${prefix}2_joint" type="revolute">
+		<joint name="${prefix}shoulder_pitch_joint" type="revolute">
 			<origin xyz="0 0 0.0265" rpy="${PI/2} 0 0" />
-			<parent link="${prefix}1_link" />
-			<child link="${prefix}2_link" />
+			<parent link="${prefix}shoulder_link" />
+			<child link="${prefix}bicep_link" />
 			<axis xyz="0 0 -1" />
-			<limit effort="3.0" velocity="6.178465545" lower="${joint_2_lower_limit}" upper="${joint_2_upper_limit}" />
-		</joint>
-		<link name="${prefix}2_link">
+			<limit effort="3.0" velocity="6.178465545" lower="${shoulder_pitch_joint_lower_limit}" upper="${shoulder_pitch_joint_upper_limit}" />
+		</joint>
+		<link name="${prefix}bicep_link">
 			<inertial>
 			  <origin xyz="-0.079312 0.00175 0.0073486" rpy="-${PI/2} 0 -${PI/2}" />
@@ -104,214 +108,188 @@
 			  </geometry>
 			</collision>
-	  </link>
-	  <!-- ELBOW -->
-	  <joint name="${prefix}3_joint" type="revolute">
-		<origin xyz="0.0385 0.1445 0.0" rpy="0 0 0" />
-		<parent link="${prefix}2_link" />
-		<child link="${prefix}3_link" />
-		<axis xyz="0 0 1" />
-		<limit
-		  effort="3.0"
-		  velocity="6.178465545"
-		  lower="${joint_3_lower_limit}"
-		  upper="${joint_3_upper_limit}"/>
-	  </joint>
-	  <link name="${prefix}3_link">
-		<inertial>
-		  <origin xyz="0.0851888339312843 0.00136288621406396 -0.000141576344087929" rpy="-${PI/2} 0 0" />
-		  <mass value="0.138705662443181" />
-		  <inertia  ixx="9.73074886909647E-05" ixy="-2.7259894490049E-06" ixz="8.2757647661483E-07"
-					iyy="0.000291190570207828" iyz="-7.99252279784603E-09"
-					izz="0.000367301178753318" />
-		</inertial>
-		<visual>
-		  <origin xyz="0 0 0" rpy="-${PI/2} 0 0" />
-		  <geometry>
-			<mesh filename="package://phantomx_reactor_arm_description/meshes/forearm_link.STL" />
-		  </geometry>
-		  <material name="">
-			<color rgba="0.25098 0.25098 0.25098 1" />
-		  </material>
-		</visual>
-		<collision>
-		  <origin xyz="0 0 0" rpy="-${PI/2} 0 0" />
-		  <geometry>
-			<mesh
-			  filename="package://phantomx_reactor_arm_description/meshes/forearm_link_hull.STL" />
-		  </geometry>
-		</collision>
-	  </link>
-	  <!-- WRIST PITCH -->
-	  <joint name="${prefix}4_joint" type="revolute">
-		<origin xyz="0.1535 0 0" rpy="0 0 0" />
-		<parent link="${prefix}3_link" />
-		<child link="${prefix}4_link" />
-		<axis xyz="0 0 1" />
-		<limit effort="1.5" velocity="6.178465545" lower="${joint_4_lower_limit}" upper="${joint_4_upper_limit}" />
-	  </joint>
-	  <link name="${prefix}4_link">
-		<inertial>
-		  <origin xyz="0.0426453655090486 0.0017494960392062 0.00984847105297723" rpy="-${PI/2} 0 0" />
-		  <mass value="0.0605067986491363" />
-		  <inertia  ixx="1.78648656995261E-05" ixy="1.11621731933541E-10" ixz="3.58888722407994E-06"
-					iyy="2.8352036542644E-05" iyz="-2.18072661043818E-10"
-					izz="2.38673851634115E-05" />
-		</inertial>
-		<visual>
-		  <origin xyz="0 0 0" rpy="-${PI/2} 0 0" />
-		  <geometry>
-			<mesh filename="package://phantomx_reactor_arm_description/meshes/wrist_1.STL" />
-		  </geometry>
-		  <material name="">
-			<color rgba="0.25098 0.25098 0.25098 1" />
-		  </material>
-		</visual>
-		<collision>
-		  <origin xyz="0 0 0" rpy="-${PI/2} 0 0" />
-		  <geometry>
-			<mesh filename="package://phantomx_reactor_arm_description/meshes/wrist_1_hull.STL" />
-		  </geometry>
-		</collision>
-	  </link>
-	  <!-- WRIST ROLL -->
-	  <joint name="${prefix}5_joint" type="revolute">
-		<origin xyz="0.071 0.00175 0" rpy="0 0 0" />
-		<parent link="${prefix}4_link" />
-		<child link="${prefix}5_link" />
-		<axis xyz="1 0 0" />
-		<limit effort="1.5" velocity="6.178465545" lower="-3.141593" upper="3.141593" />
-	  </joint>
-	  <link	name="${prefix}5_link">
-		<inertial>
-		  <origin xyz="0.022349 -5.4754E-07 0.0089164" rpy="0 0 0" />
-		  <mass value="0.055706" />
-		  <inertia  ixx="1.5957E-05" ixy="2.0952E-10" ixz="3.3629E-06"
-					iyy="2.1196E-05" iyz="-2.4643E-10"
-					izz="1.4482E-05" />
-		</inertial>
-		<visual>
-		  <origin xyz="0 0 0" rpy="-${PI/2} 0 0" />
-		  <geometry>
-			<mesh filename="package://phantomx_reactor_arm_description/meshes/wrist_2.STL" />
-		  </geometry>
-		  <material name="">
-			<color rgba="0.25098 0.25098 0.25098 1" />
-		  </material>
-		</visual>
-		<collision>
-		  <origin xyz="0 0 0" rpy="0 0 0" />
-		  <geometry>
-			<mesh filename="package://phantomx_reactor_arm_description/meshes/wrist_2_hull.STL" />
-		  </geometry>
-		</collision>
-	  </link>
-	  <!-- GRIPPER -->
-	  <!--joint name="gripper_joint" type="fixed">
-		<origin xyz="0.04789 0 0" rpy="0 0 0" />
-		<parent link="${prefix}5_link" />
-		<child link="${prefix}gripper_link" />
-	  </joint>
-	  <link name="${prefix}gripper_link">
-		<inertial>
-		  <origin xyz="0.0091884 -7.3309E-13 -3.4513E-05" rpy="0 0 0" />
-		  <mass value="0.02487" />
-		  <inertia 	ixx="1.5997E-05" ixy="1.6551E-16" ixz="8.3911E-09"
-					iyy="7.3918E-06" iyz="-2.7145E-16"
-					izz="1.5931E-05" />
-		</inertial>
-		<visual>
-		  <origin xyz="0 0 0" rpy="${PI/2} 0 0" />
-		  <geometry>
-			<mesh filename="package://phantomx_reactor_arm_description/meshes/gripper_link.STL" />
-		  </geometry>
-		  <material name="">
-			<color rgba="0.25098 0.25098 0.25098 1" />
-		  </material>
-		</visual>
-		<collision>
-		  <origin xyz="0 0 0" rpy="0 0 0" />
-		  <geometry>
-			<mesh filename="package://phantomx_reactor_arm_description/meshes/gripper_link_hull.STL" />
-		  </geometry>
-		</collision>
-	  </link-->
-	  <joint name="${prefix}guide_joint" type="fixed">
-		<origin xyz="0.05 0.00 0"   rpy="${PI/2} 0 0" />
-		<parent link="${prefix}5_link" />
-		<child link="${prefix}gripper_link_guide" />
-		<axis xyz="0 0 1" />
-		<limit effort="1.5" velocity="6.178465545" lower="0" upper="1.57"/>
-	</joint>
-	<link name="${prefix}gripper_link_guide">
-		<inertial>
-			<origin xyz="0.0091884 -7.3309E-13 -3.4513E-05" rpy="0 0 0" />
-			<mass value="0.02487" />
-			<inertia ixx="1.5997E-05" ixy="1.6551E-16" ixz="8.3911E-09" iyy="7.3918E-06" iyz="-2.7145E-16" izz="1.5931E-05" />
-		</inertial>
-		<visual>
-			<origin xyz="0 0 0" rpy="1.57 3.14 1.57" />
-			<geometry>
-				<mesh filename="package://phantomx_reactor_arm_description/meshes/Guide_Rail_Fixed_Centered.stl" scale="0.01 0.01 0.01" />
-			</geometry>
-			<material name="">
-				<color rgba="0.25098 0.25098 0.25098 1" />
-			</material>
-		</visual>
-		<collision>
-			<origin xyz="0 0 0" rpy="1.57 3.14 1.57" />
-			<geometry>
-				<mesh filename="package://phantomx_reactor_arm_description/meshes/Guide_Rail_Fixed_Centered.stl" scale="0.01 0.01 0.01" />
-			</geometry>
-		</collision>
-	</link>
-	<joint name="${prefix}gripper_joint" type="prismatic">
-		<origin xyz="0.0202 0.030 0"   rpy="0 0 0" />
-		<parent link="${prefix}gripper_link_guide" />
-		<child link="${prefix}gripper_link_right" />
-		<axis xyz="0 -0.00900 0" />
-		<limit effort="1.5" velocity="6.178465545" lower="0" upper="1.9" />
-	</joint>
-	<link name="${prefix}gripper_link_right">
-		<visual>
-			<origin xyz="0 0.00 0" rpy="-1.57 -1.57 0" />
-			<geometry>
-				<mesh filename="package://phantomx_reactor_arm_description/meshes/Gripper_Hand_Fixed_Centered.stl" scale="0.01 0.01 0.01" />
-			</geometry>
-			<material name="">
-				<color rgba="0.25098 0.25098 0.25098 1" />
-			</material>
-		</visual>
-		<collision>
-			<origin xyz="0 0.0 0" rpy="-1.57 -1.57 0" />
-			<geometry>
-				<mesh filename="package://phantomx_reactor_arm_description/meshes/Gripper_Hand_Fixed_Centered.stl" scale="0.01 0.01 0.01" />
-			</geometry>
-		</collision>
-	</link>
-	<joint name="${prefix}gripper_joint_left" type="prismatic">
-		<origin xyz="0.0202 -0.030 0" rpy="0 0 0" />
-		<parent link="${prefix}gripper_link_guide" />
-		<child link="${prefix}gripper_link_left" />
-		<axis xyz="0 -0.00900 0" />
-		<limit effort="1.5" velocity="6.178465545"  lower="-1.9" upper="0" />
-		<mimic joint="${prefix}gripper_joint" multiplier="-1.0"/>
-	</joint>
-	<link name="${prefix}gripper_link_left">
-		<visual>
-			<origin xyz="0 0 0" rpy="1.57 1.57 0" />
-			<geometry>
-				<mesh filename="package://phantomx_reactor_arm_description/meshes/Gripper_Hand_Fixed_Centered.stl" scale="0.01 0.01 0.01" />
-			</geometry>
-			<material name="">
-				<color rgba="0.25098 0.25098 0.25098 1" />
-			</material>
-		</visual>
-		<collision>
-			<origin xyz="0 0.0 0" rpy="1.57 1.57 0" />
-			<geometry>
-				<mesh filename="package://phantomx_reactor_arm_description/meshes/Gripper_Hand_Fixed_Centered.stl" scale="0.01 0.01 0.01" />
-			</geometry>
-		</collision>
-	</link>
+		</link>
+	    <!-- ELBOW PITCH-->
+		<joint name="${prefix}elbow_pitch_joint" type="revolute">
+			<origin xyz="0.0385 0.1445 0" rpy="-${PI/2} 0 0" />
+			<parent link="${prefix}bicep_link" />
+			<child link="${prefix}forearm_link" />
+			<axis xyz="0 1 0" /> <limit effort="3.0" velocity="6.178465545" lower="${elbow_pitch_joint_lower_limit}" upper="${elbow_pitch_joint_upper_limit}" />
+		</joint>
+		<link name="${prefix}forearm_link">
+			<inertial>
+				<origin xyz="0.0851888339312843 0.00136288621406396 -0.000141576344087929" rpy="0 0 0" />
+				<mass value="0.138705662443181" />
+				<inertia 	ixx="9.73074886909647E-05" ixy="-2.7259894490049E-06" ixz="8.2757647661483E-07"
+							iyy="0.000291190570207828" iyz="-7.99252279784603E-09"
+							izz="0.000367301178753318" />
+			</inertial>
+			<visual>
+				<origin xyz="0 0 0" rpy="0 0 0" />
+				<geometry>
+					<mesh filename="package://phantomx_reactor_arm_description/meshes/forearm_link.STL" />
+				</geometry>
+				<material name="">
+					<color rgba="0.25098 0.25098 0.25098 1" />
+				</material>
+			</visual>
+			<collision>
+				<origin xyz="0 0 0" rpy="0 0 0" />
+				<geometry>
+					<mesh filename="package://phantomx_reactor_arm_description/meshes/forearm_link_hull.STL" />
+				</geometry>
+			</collision>
+		</link>
+		<!-- WRIST PITCH-->
+		<joint name="${prefix}wrist_pitch_joint" type="revolute">
+			<origin xyz="0.1535 0 0"   rpy="0 0 0" />
+			<parent link="${prefix}forearm_link" />
+			<child link="${prefix}wrist_1_link" />
+			<axis xyz="0 1 0" />
+			<limit effort="1.5" velocity="6.178465545" lower="${wrist_pitch_lower_limit}" upper="${wrist_pitch_upper_limit}"/>
+		</joint>
+		<link name="${prefix}wrist_1_link">
+			<inertial>
+				<origin xyz="0.0426453655090486 0.0017494960392062 0.00984847105297723" rpy="0 0 0" />
+				<mass value="0.0605067986491363" />
+				<inertia 	ixx="1.78648656995261E-05" ixy="1.11621731933541E-10" ixz="3.58888722407994E-06"
+							iyy="2.8352036542644E-05" iyz="-2.18072661043818E-10"
+							izz="2.38673851634115E-05" />
+			</inertial>
+			<visual>
+				<origin xyz="0 0 0" rpy="0 0 0" />
+				<geometry>
+					<mesh filename="package://phantomx_reactor_arm_description/meshes/wrist_1.STL" />
+				</geometry>
+				<material name="">
+					<color rgba="0.25098 0.25098 0.25098 1" />
+				</material>
+			</visual>
+			<collision>
+				<origin xyz="0 0 0" rpy="0 0 0" />
+				<geometry>
+					<mesh filename="package://phantomx_reactor_arm_description/meshes/wrist_1_hull.STL" />
+				</geometry>
+			</collision>
+		</link>
+		<!-- WRIST ROLL -->
+		<joint name="${prefix}wrist_roll_joint" type="revolute">
+			<origin xyz="0.071 0.00175 0" rpy="0 0 0" />
+			<parent link="${prefix}wrist_1_link" />
+			<child link="${prefix}wrist_2_link" />
+			<axis xyz="1 0 0" />
+			<limit effort="1.5" velocity="6.178465545" lower="${wrist_roll_lower_limit}" upper="${wrist_roll_upper_limit}" />
+		</joint>
+		<link name="${prefix}wrist_2_link">
+			<inertial>
+				<origin xyz="0.022349 -5.4754E-07 0.0089164" rpy="0 0 0" />
+				<mass value="0.055706" />
+				<inertia 	ixx="1.5957E-05" ixy="2.0952E-10" ixz="3.3629E-06"
+							iyy="2.1196E-05" iyz="-2.4643E-10"
+							izz="1.4482E-05" />
+			</inertial>
+			<visual>
+				<origin xyz="0 0 0" rpy="0 0 0" />
+				<geometry>
+					<mesh filename="package://phantomx_reactor_arm_description/meshes/wrist_2.STL" />
+				</geometry>
+				<material name="">
+					<color rgba="0.25098 0.25098 0.25098 1" />
+				</material>
+			</visual>
+			<collision>
+				<origin xyz="0 0 0" rpy="0 0 0" />
+				<geometry>
+					<mesh filename="package://phantomx_reactor_arm_description/meshes/wrist_2_hull.STL" />
+				</geometry>
+			</collision>
+		</link>
+		<!-- GRIPPER -->
+		<joint name="${prefix}gripper_guide_joint" type="fixed">
+			<origin xyz="0.05 0.00 0"   rpy="0 0 0" />
+			<parent link="${prefix}wrist_2_link" />
+			<child link="${prefix}gripper_guide_link" />
+			<axis xyz="0 0 1" />
+			<limit effort="1.5" velocity="6.178465545" lower="0" upper="1.57"/>
+		</joint>
+		<link name="${prefix}gripper_guide_link">
+			<inertial>
+				<origin xyz="0.0091884 -7.3309E-13 -3.4513E-05" rpy="0 0 0" />
+				<mass value="0.02487" />
+				<inertia ixx="1.5997E-05" ixy="1.6551E-16" ixz="8.3911E-09" iyy="7.3918E-06" iyz="-2.7145E-16" izz="1.5931E-05" />
+			</inertial>
+			<visual>
+				<origin xyz="0 0 0" rpy="1.57 3.14 1.57" />
+				<geometry>
+					<mesh filename="package://phantomx_reactor_arm_description/meshes/Guide_Rail_Fixed_Centered.stl" scale="0.01 0.01 0.01" />
+				</geometry>
+				<material name="">
+					<color rgba="0.25098 0.25098 0.25098 1" />
+				</material>
+			</visual>
+			<collision>
+				<origin xyz="0 0 0" rpy="1.57 3.14 1.57" />
+				<geometry>
+					<mesh filename="package://phantomx_reactor_arm_description/meshes/Guide_Rail_Fixed_Centered.stl" scale="0.01 0.01 0.01" />
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