Commit message: MOD: Tested dynamixel moveit and controller OK

File: phantomx_reactor_arm_description/urdf/phantomx_reactor_wrist_gripper.urdf.xacro (robot description, xacro)
@@ -3,483 +3,258 @@
 <!-- Original from https://github.com/a-price/reactor_description/ -->
 <!-- Modified by Samir Parikh (sdparikh at gmail dot com) for movable gripper functionality -->
-<robot
-name="phantomx_reactor_arm_description"
-xmlns:xacro="http://ros.org/wiki/xacro">
-<link
-name="base_link">
-<inertial>
-  <origin
-    xyz="-3.9657E-09 2.0144E-09 0.04262"
-    rpy="0 0 0" />
-  <mass
-    value="0.33742" />
-  <inertia
-    ixx="0.0011303"
-    ixy="2.3398E-15"
-    ixz="5.3844E-11"
-    iyy="0.0011303"
-    iyz="-2.735E-11"
-    izz="0.0016747" />
-</inertial>
-<visual>
-  <origin
-    xyz="0 0 0"
-    rpy="0 0 0" />
-  <geometry>
-    <mesh
-      filename="package://phantomx_reactor_arm_description/meshes/base_link.STL" />
-  </geometry>
-  <material
-    name="">
-    <color
-      rgba="0.25098 0.25098 0.25098 1" />
-  </material>
-</visual>
-<collision>
-  <origin
-    xyz="0 0 0"
-    rpy="0 0 0" />
-  <geometry>
-    <mesh
-      filename="package://phantomx_reactor_arm_description/meshes/base_link_hull.STL" />
-  </geometry>
-</collision>
-</link>
-<link
-name="shoulder_link">
-<inertial>
-  <origin
-    xyz="5.5296E-07 0.00048339 0.0026355"
-    rpy="0 0 0" />
-  <mass
-    value="0.069055" />
-  <inertia
-    ixx="7.786E-05"
-    ixy="4.5909E-11"
-    ixz="-6.4873E-11"
-    iyy="4.1745E-05"
-    iyz="2.8244E-07"
-    izz="0.0001073" />
-</inertial>
-<visual>
-  <origin
-    xyz="0 0 0"
-    rpy="0 0 0" />
-  <geometry>
-    <mesh
-      filename="package://phantomx_reactor_arm_description/meshes/shoulder_link.STL" />
-  </geometry>
-  <material
-    name="">
-    <color
-      rgba="0.25098 0.25098 0.25098 1" />
-  </material>
-</visual>
-<collision>
-  <origin
-    xyz="0 0 0"
-    rpy="0 0 0" />
-  <geometry>
-    <mesh
-      filename="package://phantomx_reactor_arm_description/meshes/shoulder_link_hull.STL" />
-  </geometry>
-</collision>
-</link>
-<joint
-name="shoulder_yaw"
-type="revolute">
-<origin
-  xyz="0 0 0.090"
-  rpy="0 0 0" />
-<parent
-  link="base_link" />
-<child
-  link="shoulder_link" />
-<axis
-  xyz="0 0 1" />
-<limit
-  effort="1.5"
-  velocity="6.178465545"
-  lower="-2.57079632679"
-  upper="2.57079632679" />
-</joint>
-<link
-name="bicep_link">
-<inertial>
-  <origin
-    xyz="-0.079312 0.00175 0.0073486"
-    rpy="0 0 0" />
-  <mass
-    value="0.29331" />
-  <inertia
-    ixx="0.00040741"
-    ixy="-1.1578E-09"
-    ixz="-0.00014106"
-    iyy="0.0010604"
-    iyz="1.1578E-09"
-    izz="0.0012838" />
-</inertial>
-<visual>
-  <origin
-    xyz="0 0 0"
-    rpy="0 0 0" />
-  <geometry>
-    <mesh
-      filename="package://phantomx_reactor_arm_description/meshes/bicep_link.STL" />
-  </geometry>
-  <material
-    name="">
-    <color
-      rgba="0.25098 0.25098 0.25098 1" />
-  </material>
-</visual>
-<collision>
-  <origin
-    xyz="0 0 0"
-    rpy="0 0 0" />
-  <geometry>
-    <mesh
-      filename="package://phantomx_reactor_arm_description/meshes/bicep_link_hull.STL" />
-  </geometry>
-</collision>
-</link>
-<joint
-name="shoulder_pitch"
-type="revolute">
-<origin
-  xyz="0 0 0.0265"
-  rpy="0 1.57 0" />
-<parent
-  link="shoulder_link" />
-<child
-  link="bicep_link" />
-<axis
-  xyz="0 1 0" />
-<limit
-  effort="3.0"
-  velocity="6.178465545"
-  lower="-1.7079632679"
-  upper="1.57079632679" />
-</joint>
-<link
-name="forearm_link">
-<inertial>
-  <origin
-    xyz="0.0851888339312843 0.00136288621406396 -0.000141576344087929"
-    rpy="0 0 0" />
-  <mass
-    value="0.138705662443181" />
-  <inertia
-    ixx="9.73074886909647E-05"
-    ixy="-2.7259894490049E-06"
-    ixz="8.2757647661483E-07"
-    iyy="0.000291190570207828"
-    iyz="-7.99252279784603E-09"
-    izz="0.000367301178753318" />
-</inertial>
-<visual>
-  <origin
-    xyz="0 0 0"
-    rpy="0 0 0" />
-  <geometry>
-    <mesh
-      filename="package://phantomx_reactor_arm_description/meshes/forearm_link.STL" />
-  </geometry>
-  <material
-    name="">
-    <color
-      rgba="0.25098 0.25098 0.25098 1" />
-  </material>
-</visual>
-<collision>
-  <origin
-    xyz="0 0 0"
-    rpy="0 0 0" />
-  <geometry>
-    <mesh
-      filename="package://phantomx_reactor_arm_description/meshes/forearm_link_hull.STL" />
-  </geometry>
-</collision>
-</link>
-<joint
-name="elbow_pitch"
-type="revolute">
-<origin
-  xyz="-0.1445 0 0.0385"
-  rpy="0 -1.57079632679 0" />
-<parent
-  link="bicep_link" />
-<child
-  link="forearm_link" />
-<axis
-  xyz="0 1 0" />
-<limit
-  effort="3.0"
-  velocity="6.178465545"
-  lower="-1.57079632679"
-  upper="1.57079632679" />
-</joint>
-<link
-name="wrist_1">
-<inertial>
-  <origin
-    xyz="0.0426453655090486 0.0017494960392062 0.00984847105297723"
-    rpy="0 0 0" />
-  <mass
-    value="0.0605067986491363" />
-  <inertia
-    ixx="1.78648656995261E-05"
-    ixy="1.11621731933541E-10"
-    ixz="3.58888722407994E-06"
-    iyy="2.8352036542644E-05"
-    iyz="-2.18072661043818E-10"
-    izz="2.38673851634115E-05" />
-</inertial>
-<visual>
-  <origin
-    xyz="0 0 0"
-    rpy="0 0 0" />
-  <geometry>
-    <mesh
-      filename="package://phantomx_reactor_arm_description/meshes/wrist_1.STL" />
-  </geometry>
-  <material
-    name="">
-    <color
-      rgba="0.25098 0.25098 0.25098 1" />
-  </material>
-</visual>
-<collision>
-  <origin
-    xyz="0 0 0"
-    rpy="0 0 0" />
-  <geometry>
-    <mesh
-      filename="package://phantomx_reactor_arm_description/meshes/wrist_1_hull.STL" />
-  </geometry>
-</collision>
-</link>
-<joint
-name="wrist_pitch"
-type="revolute">
-<origin
-  xyz="0.1535 0 0"
-  rpy="0 0 0" />
-<parent
-  link="forearm_link" />
-<child
-  link="wrist_1" />
-<axis
-  xyz="0 1 0" />
-<limit
-  effort="1.5"
-  velocity="6.178465545"
-  lower="-1.7"
-  upper="1.9" />
-</joint>
-<link
-name="wrist_2">
-<inertial>
-  <origin
-    xyz="0.022349 -5.4754E-07 0.0089164"
-    rpy="0 0 0" />
-  <mass
-    value="0.055706" />
-  <inertia
-    ixx="1.5957E-05"
-    ixy="2.0952E-10"
-    ixz="3.3629E-06"
-    iyy="2.1196E-05"
-    iyz="-2.4643E-10"
-    izz="1.4482E-05" />
-</inertial>
-<visual>
-  <origin
-    xyz="0 0 0"
-    rpy="0 0 0" />
-  <geometry>
-    <mesh
-      filename="package://phantomx_reactor_arm_description/meshes/wrist_2.STL" />
-  </geometry>
-  <material
-    name="">
-    <color
-      rgba="0.25098 0.25098 0.25098 1" />
-  </material>
-</visual>
-<collision>
-  <origin
-    xyz="0 0 0"
-    rpy="0 0 0" />
-  <geometry>
-    <mesh
-      filename="package://phantomx_reactor_arm_description/meshes/wrist_2_hull.STL" />
-  </geometry>
-</collision>
-</link>
-<joint
-name="wrist_roll"
-type="revolute">
-<origin
-  xyz="0.071 0.00175 0"
-  rpy="0 0 0" />
-<parent
-  link="wrist_1" />
-<child
-  link="wrist_2" />
-<axis
-  xyz="1 0 0" />
-<limit
-  effort="1.5"
-  velocity="6.178465545"
-  lower="-3.141593"
-  upper="3.141593" />
-</joint>
-<link
-name="gripper_link_guide">
-<inertial>
-  <origin
-    xyz="0.0091884 -7.3309E-13 -3.4513E-05"
-    rpy="0 0 0" />
-  <mass
-    value="0.02487" />
-  <inertia
-    ixx="1.5997E-05"
-    ixy="1.6551E-16"
-    ixz="8.3911E-09"
-    iyy="7.3918E-06"
-    iyz="-2.7145E-16"
-    izz="1.5931E-05" />
-</inertial>
-<visual>
-  <origin
-    xyz="0 0 0"
-    rpy="1.57 3.14 1.57" />
-  <geometry>
-    <mesh
-      filename="package://phantomx_reactor_arm_description/meshes/Guide_Rail_Fixed_Centered.stl" scale="0.01 0.01 0.01" />
-  </geometry>
-  <material
-    name="">
-    <color
-      rgba="0.25098 0.25098 0.25098 1" />
-  </material>
-</visual>
-<collision>
-  <origin
-    xyz="0 0 0"
-    rpy="1.57 3.14 1.57" />
-  <geometry>
-    <mesh
-      filename="package://phantomx_reactor_arm_description/meshes/Guide_Rail_Fixed_Centered.stl" scale="0.01 0.01 0.01" />
-  </geometry>
-</collision>
-</link>
-<joint
-name="guide_joint"
-type="fixed">
-<origin
-  xyz="0.05 0.00 0"
-  rpy="0 0 0" />
-<parent
-  link="wrist_2" />
-<child
-  link="gripper_link_guide" />
-<axis
-  xyz="0 0 1" />
-<limit
-  effort="1.5"
-  velocity="6.178465545"
-  lower="0"
-  upper="1.57" />
-</joint>
-<link
-name="gripper_link_right">
-<visual>
-  <origin
-    xyz="0 0.00 0"
-    rpy="-1.57 -1.57 0" />
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
File: phantomx_reactor_arm_description/urdf/phantomx_reactor_wrist_unified.urdf.xacro (robot description, xacro)
@@ -41,14 +41,15 @@
 			</collision>
 		</link>
-		<!-- SHOULDER YAW -->
-		<joint name="${prefix}1_joint" type="revolute">
+		<!-- SHOULDER PAN -->
+		<joint name="${prefix}shoulder_yaw" type="revolute">
 			<origin xyz="0 0 0.081" rpy="0 0 0" />
+			<!--origin xyz="0 0 0.081" rpy="0 0 0" /-->
 			<parent link="${prefix}base_link" />
-			<child link="${prefix}1_link" />
+			<child link="${prefix}shoulder_link" />
 			<axis xyz="0 0 1" />
 			<limit effort="1.5" velocity="6.178465545" lower="-3.141593" upper="3.141593" />
 			<!--limit effort="1.5" velocity="6.178465545" lower="-2.57079632679" upper="2.57079632679" /-->
 		</joint>
-		<link name="${prefix}1_link">
+		<link name="${prefix}shoulder_link">
 			<inertial>
 			  <origin xyz="5.5296E-07 0.00048339 0.0026355" rpy="0 0 0" />
@@ -73,13 +74,13 @@
 			</collision>
 		</link>
-		<!-- SHOULDER PITCH -->
-		<joint name="${prefix}2_joint" type="revolute">
+		<!-- SHOULDER TILT -->
+		<joint name="${prefix}shoulder_pitch" type="revolute">
 			<origin xyz="0 0 0.0265" rpy="${PI/2} 0 0" />
-			<parent link="${prefix}1_link" />
-			<child link="${prefix}2_link" />
+			<parent link="${prefix}shoulder_link" />
+			<child link="${prefix}bicep_link" />
 			<axis xyz="0 0 -1" />
 			<limit effort="3.0" velocity="6.178465545" lower="${joint_2_lower_limit}" upper="${joint_2_upper_limit}" />
 		</joint>
-		<link name="${prefix}2_link">
+		<link name="${prefix}bicep_link">
 			<inertial>
 			  <origin xyz="-0.079312 0.00175 0.0073486" rpy="-${PI/2} 0 -${PI/2}" />
@@ -142,6 +143,6 @@
 		</collision>
 	  </link>
-	  <!-- WRIST PITCH -->
-	  <joint name="${prefix}4_joint" type="revolute">
+	  <!-- WRIST TILT -->
+	  <joint name="${prefix}4_joint"	type="revolute">
 		<origin xyz="0.1535 0 0" rpy="0 0 0" />
 		<parent link="${prefix}3_link" />
@@ -174,5 +175,5 @@
 		</collision>
 	  </link>
-	  <!-- WRIST ROLL -->
+	  <!-- WRIST ROTATION -->
 	  <joint name="${prefix}5_joint" type="revolute">
 		<origin xyz="0.071 0.00175 0" rpy="0 0 0" />
@@ -207,5 +208,5 @@
 	  </link>
 	  <!-- GRIPPER -->
-	  <!--joint name="gripper_joint" type="fixed">
+	  <!--joint name="${prefix}gripper_joint" type="fixed">
 		<origin xyz="0.04789 0 0" rpy="0 0 0" />
 		<parent link="${prefix}5_link" />
@@ -236,12 +237,12 @@
 		</collision>
 	  </link-->
-	  <joint name="${prefix}guide_joint" type="fixed">
-		<origin xyz="0.05 0.00 0"   rpy="${PI/2} 0 0" />
+	  <joint name="guide_joint" type="fixed">
+		<origin xyz="0.05 0.00 0"   rpy="0 0 0" />
 		<parent link="${prefix}5_link" />
-		<child link="${prefix}gripper_link_guide" />
+		<child link="gripper_link_guide" />
 		<axis xyz="0 0 1" />
 		<limit effort="1.5" velocity="6.178465545" lower="0" upper="1.57"/>
 	</joint>
-	<link name="${prefix}gripper_link_guide">
+	<link name="gripper_link_guide">
 		<inertial>
 			<origin xyz="0.0091884 -7.3309E-13 -3.4513E-05" rpy="0 0 0" />
@@ -265,12 +266,12 @@
 		</collision>
 	</link>
-	<joint name="${prefix}gripper_joint" type="prismatic">
+	<joint name="gripper_joint" type="prismatic">
 		<origin xyz="0.0202 0.030 0"   rpy="0 0 0" />
-		<parent link="${prefix}gripper_link_guide" />
-		<child link="${prefix}gripper_link_right" />
+		<parent link="gripper_link_guide" />
+		<child link="gripper_link_right" />
 		<axis xyz="0 -0.00900 0" />
 		<limit effort="1.5" velocity="6.178465545" lower="0" upper="1.9" />
 	</joint>
-	<link name="${prefix}gripper_link_right">
+	<link name="gripper_link_right">
 		<visual>
 			<origin xyz="0 0.00 0" rpy="-1.57 -1.57 0" />
@@ -289,13 +290,13 @@
 		</collision>
 	</link>
-	<joint name="${prefix}gripper_joint_left" type="prismatic">
+	<joint name="gripper_joint_left" type="prismatic">
 		<origin xyz="0.0202 -0.030 0" rpy="0 0 0" />
-		<parent link="${prefix}gripper_link_guide" />
-		<child link="${prefix}gripper_link_left" />
+		<parent link="gripper_link_guide" />
+		<child link="gripper_link_left" />
 		<axis xyz="0 -0.00900 0" />
 		<limit effort="1.5" velocity="6.178465545"  lower="-1.9" upper="0" />
-		<mimic joint="${prefix}gripper_joint" multiplier="-1.0"/>
+		<mimic joint="gripper_joint" multiplier="-1.0"/>
 	</joint>
-	<link name="${prefix}gripper_link_left">
+	<link name="gripper_link_left">
 		<visual>
 			<origin xyz="0 0 0" rpy="1.57 1.57 0" />
